File: dc_receiver/dc_receiver.kicad_pcb (KiCad board)
At the start: 2 copper layers, 83 x 30 mm, 62 parts, among them J1 Conn_01x02, J2 Conn_01x02, J3 Conn_01x02, J4 Conn_01x02, J5 HOLE, J6 HOLE, J7 HOLE, J8 HOLE, Q1 BC548, Q2 BC548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

Commit message: add renders, pdf schematic, ready for export
Routing:
- added copper zone on B.Cu, net GND
Other:
- board text added: "+"
- board text added: "+12V"
- board text added: "AUDIO OUT"
- board text added: "LO"
- board text added: "RF IN"
