File: dc_receiver/dc_receiver.sch (KiCad schematic (older format))
At the start: 58 parts

Commit message: finish schenmatic add layout
Parts:
- removed C?: 100u, symbol Device:C_Small
- added C3: 100n, Capacitor_SMD:C_1206_3216Metric_Pad1.42x1.75mm_HandSolder, symbol Device:C_Small
- added J5, J6, J7, J8: HOLE, dc_receiver:HOLE, symbol Connector_Generic:Conn_01x01
- C1, C13, C17, C19, C2, C20, C21, C22, C23, C7, C8: renamed from C?; footprint (none) -> Capacitor_SMD:C_1206_3216Metric_Pad1.42x1.75mm_HandSolder
- C10, C11, C14, C16, C5: renamed from C?; footprint (none) -> Capacitor_THT:CP_Radial_D6.3mm_P2.50mm
- C12, C18, C6: renamed from C?; footprint (none) -> Capacitor_THT:CP_Radial_D5.0mm_P2.00mm
- C15: renamed from C?; footprint (none) -> Capacitor_THT:CP_Radial_D8.0mm_P3.50mm
- C9: renamed from C?; value 47u -> 100u; footprint (none) -> Capacitor_THT:CP_Radial_D8.0mm_P3.50mm
- J1, J2, J3, J4: renamed from J?; footprint (none) -> Connector_PinHeader_2.54mm:PinHeader_1x02_P2.54mm_Vertical
- L1: renamed from L?; footprint (none) -> dc_receiver:ft37-43-choke
- Q1, Q2, Q3, Q4: renamed from Q?; footprint Package_TO_SOT_THT:TO-92_Inline -> Package_TO_SOT_THT:TO-92_Inline_Wide
- R1, R10, R11, R12, R13, R14, R15, R16, R17, R18, R19, R2, R20, R21, R22, R23, R24, R3, R4, R5, R6, R7, R8, R9: renamed from R?; footprint (none) -> Resistor_SMD:R_1206_3216Metric_Pad1.42x1.75mm_HandSolder
- RV1: renamed from RV?; footprint (none) -> Connector_PinHeader_2.54mm:PinHeader_1x03_P2.54mm_Vertical
- U1: renamed from U?; footprint (none) -> dc_receiver:ERMS-1
- U2: renamed from U?; footprint (none) -> Package_SO:SO-8_3.9x4.9mm_P1.27mm
Connections:
- net AUDIO_OUT: now also C15.2; no longer C15.1
- net GND: now also C12.2, C9.2, J5.1 (Pin_1), J6.1 (Pin_1), J7.1 (Pin_1), J8.1 (Pin_1); no longer C12.1, C9.1
- net RF: now also C3.2; no longer U1.4 (RF)
- net at R15.1, U2.5: now also C15.1; no longer C15.2
- net at R12.2, U2.6 (V+): now also C9.1; no longer C9.2
- net at U2.7 (BYPASS): now also C12.1; no longer C12.2
- new net: C3.1, U1.4 (RF)

Commit message: add renders, pdf schematic, ready for export
Other:
- note added: "DIPLEXER"
- note added: "GAIN BLOCK 1"
- note added: "GAIN BLOCK 2"
- note added: "GAIN BLOCK 3"
- note added: "LO MATCH AND PAD"
- note added: "RF MIXER TO AUDIO"
- note added: "SPEAKER AMP"
- note added: "SSB / CW BAND-PASS\nEXPERIMENT AREA"
- moved on the sheet: C10, C11, C12, C13, C14, C15, C16, C17, C18, C19, C2, C20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
